File: Fuente/Fuente.kicad_sch (KiCad schematic)
At the start: 16 parts, among them J1 USB_B_Mini, J2 Conn_01x02_Pin, J3 Conn_01x02_Pin, U2 LM1117DT-3.3, U3 TPS61087DSCR

Commit message: FootPrint modificada en el convertidor a 12v
Parts:
- U3: footprint Package_TO_SOT_SMD:TO-252-3_TabPin2 -> TPS61087DRC:IC_TPS61087DSCR
Changed lines of the file:
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@@
 			)
 		)
-		(property "Footprint" "Package_TO_SOT_SMD:TO-252-3_TabPin2"
+		(property "Footprint" "TPS61087DRC:IC_TPS61087DSCR"
 			(at 154.94 48.26 0)
 			(hide yes)

Commit message: Incorporación de agujeros de montaje y acomodo del diseño de la PCB
Parts:
- added H1, H2, H3, H4: MountingHole_Pad_MP, MountingHole:MountingHole_3mm_Pad, symbol Mechanical:MountingHole_Pad_MP
Connections:
- net GND: now also H1.MP, H2.MP, H3.MP, H4.MP

Commit message: Versión mejorada con agujeros pasantes
Parts:
- J2, J3: footprint TerminalBlock_CUI:TerminalBlock_CUI_TB007-508-02_1x02_P5.08mm_Horizontal -> TerminalBlock_Phoenix:TerminalBlock_Phoenix_MKDS-1,5-2_1x02_P5.00mm_Horizontal
Changed lines of the file:
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@@
 			)
 		)
-		(property "Footprint" "TerminalBlock_CUI:TerminalBlock_CUI_TB007-508-02_1x02_P5.08mm_Horizontal"
+		(property "Footprint" "TerminalBlock_Phoenix:TerminalBlock_Phoenix_MKDS-1,5-2_1x02_P5.00mm_Horizontal"
 			(at 49.53 24.13 0)
 			(hide yes)
@@
 			)
 		)
-		(property "Footprint" "TerminalBlock_CUI:TerminalBlock_CUI_TB007-508-02_1x02_P5.08mm_Horizontal"
+		(property "Footprint" "TerminalBlock_Phoenix:TerminalBlock_Phoenix_MKDS-1,5-2_1x02_P5.00mm_Horizontal"
 			(at 49.53 40.64 0)
 			(hide yes)
